Commit message: my_robot.xacro Left Wheel
Added the left wheel and associated joint to the my_robot.xacro file.

File: src/my_robot/urdf/my_robot.xacro (robot description, xacro)
@@ -55,3 +55,34 @@
     </visual>
   </link>
+  <link name='left_wheel'>
+    <inertial>
+      <mass value="5.0"/>
+      <origin xyz="0.0 0 0" rpy=" 0  1.5707  1.5707"/>
+      <inertia
+          ixx="0.1" ixy="0" ixz="0"
+          iyy="0.1" iyz="0"
+          izz="0.1"
+      />
+    </inertial>
+    <collision name='left_wheel_collision'>
+      <origin xyz="0.0 0 0" rpy=" 0  1.5707  1.5707"/>
+      <geometry>
+        <cylinder size="0.1 0.05"/>
+      </geometry>
+    </collision>
+    <visual name='left_wheel_visual'>
+      <origin xyz="0.0 0 0" rpy=" 0  1.5707  1.5707"/>
+      <geometry>
+        <cylinder size="0.1 0.05"/>
+      </geometry>
+    </visual>
+  </link>
+  <joint type="continuous" name="left_wheel_hinge">
+    <origin xyz="0 0.15 0" rpy="0 0 0"/>
+    <child link="left_wheel"/>
+    <parent link="chassis"/>
+    <axis xyz="0 1 0" rpy="0 0 0"/>
+    <limit effort="10000" velocity="1000"/>
+    <dynamics damping="1.0" friction="1.0"/>
+  </joint>
 </robot>

Commit message: my_robot.xacro right wheel update
Added the right wheel link and associated joint to the my_robot xacro file

File: src/my_robot/urdf/my_robot.xacro (robot description, xacro)
@@ -86,3 +86,34 @@
     <dynamics damping="1.0" friction="1.0"/>
   </joint>
+  <link name='right_wheel'>
+    <inertial>
+      <mass value="5.0"/>
+      <origin xyz="0.0 0 0" rpy=" 0  1.5707  1.5707"/>
+      <inertia
+          ixx="0.1" ixy="0" ixz="0"
+          iyy="0.1" iyz="0"
+          izz="0.1"
+      />
+    </inertial>
+    <collision name='right_wheel_collision'>
+      <origin xyz="0.0 0 0" rpy=" 0  1.5707  1.5707"/>
+      <geometry>
+        <cylinder size="0.1 0.05"/>
+      </geometry>
+    </collision>
+    <visual name='right_wheel_visual'>
+      <origin xyz="0.0 0 0" rpy=" 0  1.5707  1.5707"/>
+      <geometry>
+        <cylinder size="0.1 0.05"/>
+      </geometry>
+    </visual>
+  </link>
+  <joint type="continuous" name="right_wheel_hinge">
+    <origin xyz="0 0.15 0" rpy="0 0 0"/>
+    <child link="right_wheel"/>
+    <parent link="chassis"/>
+    <axis xyz="0 1 0" rpy="0 0 0"/>
+    <limit effort="10000" velocity="1000"/>
+    <dynamics damping="1.0" friction="1.0"/>
+  </joint>
 </robot>

Commit message: my_robot xacro camera add
Added the representative link and joint to the my_robot.xacro file.

File: src/my_robot/urdf/my_robot.xacro (robot description, xacro)
@@ -117,3 +117,35 @@
     <dynamics damping="1.0" friction="1.0"/>
   </joint>
+  <link name='camera'>
+    <pose>0 0 0 0 0 0</pose>
+    <inertial>
+      <mass value="0.1"/>
+      <origin xyz="0.05 0.05 0.05" rpy=" 0 0 0"/>
+      <inertia
+          ixx="1e-6" ixy="0" ixz="0"
+          iyy="1e-6" iyz="0"
+          izz="1e-6"
+      />
+    </inertial>
+    <collision name='camera_collision'>
+      <origin xyz="0 0 0" rpy=" 0 0 0"/>
+      <geometry>
+        <box size="0.05 0.05 0.05"/>
+      </geometry>
+    </collision>
+    <visual name='camera_visual'>
+      <origin xyz="0 0 0" rpy=" 0 0 0"/>
+      <geometry>
+        <box size="0.05 0.05 0.05"/>
+      </geometry>
+    </visual>
+    <joint type="fixed" name="camera_joint">
+    <origin xyz="0.2 0 0" rpy="0 0 0"/>
+    <child link="camera"/>
+    <parent link="chassis"/>
+    <axis xyz="0 1 0" rpy="0 0 0"/>
+    <limit effort="10000" velocity="1000"/>
+    <dynamics damping="1.0" friction="1.0"/>
+  </joint>
+  </link>
 </robot>

Commit message: my_robot.xacro hokuyo updated
Added the urdf formated links and joints representing the hokuyo LIDAR to my_robot.xacro.

File: src/my_robot/urdf/my_robot.xacro (robot description, xacro)
@@ -149,3 +149,35 @@
   </joint>
   </link>
+  <link name='hokuyo'>
+    <pose>0 0 0 0 0 0</pose>
+    <inertial>
+      <mass value="1e-5"/>
+      <origin xyz="0 0 0" rpy=" 0 0 0"/>
+      <inertia
+          ixx="1e-6" ixy="0" ixz="0"
+          iyy="1e-6" iyz="0"
+          izz="1e-6"
+      />
+    </inertial>
+    <collision name='hokuyo_collision'>
+      <origin xyz="0 0 0" rpy=" 0 0 0"/>
+      <geometry>
+        <box size="0.1 0.1 0.1"/>
+      </geometry>
+    </collision>
+    <visual name='hokuyo_visual'>
+      <origin xyz="0 0 0" rpy=" 0 0 0"/>
+      <geometry>
+        <mesh filename="package://my_robot/meshes/hokuyo.dae"/>
+      </geometry>
+    </visual>
+    <joint type="fixed" name="hokuyo_joint">
+    <origin xyz="0.15 0 0.1" rpy="0 0 0"/>
+    <child link="hokuyo"/>
+    <parent link="chassis"/>
+    <axis xyz="0 1 0" rpy="0 0 0"/>
+    <limit effort="10000" velocity="1000"/>
+    <dynamics damping="1.0" friction="1.0"/>
+  </joint>
+  </link>
 </robot>

Commit message: my_robot.xacro complete
All components of the basic my_robot model now appear in the correct places.

File: src/my_robot/urdf/my_robot.xacro (robot description, xacro)
@@ -58,5 +58,5 @@
     <inertial>
       <mass value="5.0"/>
-      <origin xyz="0.0 0 0" rpy=" 0  1.5707  1.5707"/>
+      <origin xyz="0.0 0.0 0.0" rpy="0.0 1.5707 1.5707"/>
       <inertia
           ixx="0.1" ixy="0" ixz="0"
@@ -66,13 +66,13 @@
     </inertial>
     <collision name='left_wheel_collision'>
-      <origin xyz="0.0 0 0" rpy=" 0  1.5707  1.5707"/>
+      <origin xyz="0.0 0.0 0.0" rpy="0.0 1.5707 1.5707"/>
       <geometry>
-        <cylinder size="0.1 0.05"/>
+        <cylinder length="0.05" radius="0.1"/>
       </geometry>
     </collision>
     <visual name='left_wheel_visual'>
-      <origin xyz="0.0 0 0" rpy=" 0  1.5707  1.5707"/>
+      <origin xyz="0.0 0.0 0.0" rpy="0.0 1.5707 1.5707"/>
       <geometry>
-        <cylinder size="0.1 0.05"/>
+        <cylinder length="0.05" radius="0.1"/>
       </geometry>
     </visual>
@@ -89,5 +89,5 @@
     <inertial>
       <mass value="5.0"/>
-      <origin xyz="0.0 0 0" rpy=" 0  1.5707  1.5707"/>
+      <origin xyz="0.0 0.0 0.0" rpy="0.0 1.5707 1.5707"/>
       <inertia
           ixx="0.1" ixy="0" ixz="0"
@@ -97,18 +97,18 @@
     </inertial>
     <collision name='right_wheel_collision'>
-      <origin xyz="0.0 0 0" rpy=" 0  1.5707  1.5707"/>
+      <origin xyz="0.0 0.0 0.0" rpy="0.0 1.5707 1.5707"/>
       <geometry>
-        <cylinder size="0.1 0.05"/>
+        <cylinder length="0.05" radius="0.1"/>
       </geometry>
     </collision>
     <visual name='right_wheel_visual'>
-      <origin xyz="0.0 0 0" rpy=" 0  1.5707  1.5707"/>
+      <origin xyz="0.0 0.0 0.0" rpy="0.0 1.5707 1.5707"/>
       <geometry>
-        <cylinder size="0.1 0.05"/>
+        <cylinder length="0.05" radius="0.1"/>
       </geometry>
     </visual>
   </link>
   <joint type="continuous" name="right_wheel_hinge">
-    <origin xyz="0 0.15 0" rpy="0 0 0"/>
+    <origin xyz="0 -0.15 0" rpy="0 0 0"/>
     <child link="right_wheel"/>
     <parent link="chassis"/>
@@ -118,8 +118,8 @@
   </joint>
   <link name='camera'>
-    <pose>0 0 0 0 0 0</pose>
     <inertial>
       <mass value="0.1"/>
-      <origin xyz="0.05 0.05 0.05" rpy=" 0 0 0"/>
+      <origin xyz="0.0 0.0 0.0" rpy="0.0 0.0 0.0"/>
+      <box_inertia x="0.05" y="0.05" z="0.05" m="0.1"/>
       <inertia
           ixx="1e-6" ixy="0" ixz="0"
@@ -129,5 +129,5 @@
     </inertial>
     <collision name='camera_collision'>
-      <origin xyz="0 0 0" rpy=" 0 0 0"/>
+      <origin xyz="0.0 0.0 0.0" rpy="0.0 0.0 0.0"/>
       <geometry>
         <box size="0.05 0.05 0.05"/>
@@ -135,11 +135,12 @@
     </collision>
     <visual name='camera_visual'>
-      <origin xyz="0 0 0" rpy=" 0 0 0"/>
+      <origin xyz="0.0 0.0 0.0" rpy="0.0 0.0 0.0"/>
       <geometry>
         <box size="0.05 0.05 0.05"/>
       </geometry>
     </visual>
-    <joint type="fixed" name="camera_joint">
-    <origin xyz="0.2 0 0" rpy="0 0 0"/>
+  </link>
+  <joint type="fixed" name="camera_joint">
+    <origin xyz="0.2 0.0 0.0" rpy="0 0 0"/>
     <child link="camera"/>
     <parent link="chassis"/>
@@ -148,10 +149,8 @@
     <dynamics damping="1.0" friction="1.0"/>
   </joint>
-  </link>
   <link name='hokuyo'>
-    <pose>0 0 0 0 0 0</pose>
     <inertial>
       <mass value="1e-5"/>
-      <origin xyz="0 0 0" rpy=" 0 0 0"/>
+      <origin xyz="0.0 0.0 0.0" rpy="0.0 0.0 0.0"/>
       <inertia
           ixx="1e-6" ixy="0" ixz="0"
@@ -161,5 +160,5 @@
     </inertial>
     <collision name='hokuyo_collision'>
-      <origin xyz="0 0 0" rpy=" 0 0 0"/>
+      <origin xyz="0.0 0.0 0.0" rpy="0.0 0.0 0.0"/>
       <geometry>
         <box size="0.1 0.1 0.1"/>
@@ -167,11 +166,12 @@
     </collision>
     <visual name='hokuyo_visual'>
-      <origin xyz="0 0 0" rpy=" 0 0 0"/>
+      <origin xyz="0.0 0.0 0.0" rpy="0.0 0.0 0.0"/>
       <geometry>
         <mesh filename="package://my_robot/meshes/hokuyo.dae"/>
       </geometry>
     </visual>
-    <joint type="fixed" name="hokuyo_joint">
-    <origin xyz="0.15 0 0.1" rpy="0 0 0"/>
+  </link>
+  <joint type="fixed" name="hokuyo_joint">
+    <origin xyz="0.15 0.0 0.1" rpy="0 0 0"/>
     <child link="hokuyo"/>
     <parent link="chassis"/>
@@ -180,4 +180,3 @@
     <dynamics damping="1.0" friction="1.0"/>
   </joint>
-  </link>
 </robot>

Commit message: GoChaseIt Complete
Project done with White ball Chasing Capability, Skid Steer Robot Implemented.

File: src/my_robot/urdf/my_robot.xacro (robot description, xacro)
@@ -1,3 +1,4 @@
 <?xml version='1.0'?>
+<!-- Robot Base -->
 <robot name="my_robot" xmlns:xacro="http://www.ros.org/wiki/xacro">
 <xacro:include filename="$(find my_robot)/urdf/my_robot.gazebo" />
@@ -22,5 +23,5 @@
       <origin xyz="0 0 0" rpy=" 0 0 0"/>
       <geometry>
-        <box size=".4 .2 .1"/>
+        <box size=".5 .2 .1"/>
       </geometry>
     </collision>
@@ -28,5 +29,5 @@
       <origin xyz="0 0 0" rpy=" 0 0 0"/>
       <geometry>
-        <box size=".4 .2 .1"/>
+        <box size=".5 .2 .1"/>
       </geometry>
     </visual>
@@ -56,4 +57,5 @@
     </visual>
   </link>
+  <!-- First Set of Wheels -->
   <link name='left_wheel'>
     <inertial>
@@ -80,5 +82,5 @@
   </link>
   <joint type="continuous" name="left_wheel_hinge">
-    <origin xyz="0 0.15 0" rpy="0 0 0"/>
+    <origin xyz="0.2 0.15 0" rpy="0 0 0"/>
     <child link="left_wheel"/>
     <parent link="chassis"/>
@@ -111,5 +113,5 @@
   </link>
   <joint type="continuous" name="right_wheel_hinge">
-    <origin xyz="0 -0.15 0" rpy="0 0 0"/>
+    <origin xyz="0.2 -0.15 0" rpy="0 0 0"/>
     <child link="right_wheel"/>
     <parent link="chassis"/>
@@ -118,4 +120,68 @@
     <dynamics damping="1.0" friction="1.0"/>
   </joint>
+  <!-- Second Set of Wheels -->
+  <link name='left2_wheel'>
+    <inertial>
+      <mass value="5.0"/>
+      <origin xyz="0.0 0.0 0.0" rpy="0.0 1.5707 1.5707"/>
+      <inertia
+          ixx="0.1" ixy="0" ixz="0"
+          iyy="0.1" iyz="0"
+          izz="0.1"
+      />
+    </inertial>
+    <collision name='left2_wheel_collision'>
+      <origin xyz="0.0 0.0 0.0" rpy="0.0 1.5707 1.5707"/>
+      <geometry>
+        <cylinder length="0.05" radius="0.1"/>
+      </geometry>
+    </collision>
+    <visual name='left2_wheel_visual'>
+      <origin xyz="0.0 0.0 0.0" rpy="0.0 1.5707 1.5707"/>
+      <geometry>
+        <cylinder length="0.05" radius="0.1"/>
+      </geometry>
+    </visual>
+  </link>
+  <joint type="continuous" name="left2_wheel_hinge">
+    <origin xyz="-0.25 0.15 0" rpy="0 0 0"/>
+    <child link="left2_wheel"/>
+    <parent link="chassis"/>
+    <axis xyz="0 1 0" rpy="0 0 0"/>
+    <limit effort="10000" velocity="1000"/>
+    <dynamics damping="1.0" friction="1.0"/>
+  </joint>
+  <link name='right2_wheel'>
+    <inertial>
+      <mass value="5.0"/>
+      <origin xyz="0.0 0.0 0.0" rpy="0.0 1.5707 1.5707"/>
+      <inertia
+          ixx="0.1" ixy="0" ixz="0"
+          iyy="0.1" iyz="0"
+          izz="0.1"
+      />
+    </inertial>
+    <collision name='right2_wheel_collision'>
+      <origin xyz="0.0 0.0 0.0" rpy="0.0 1.5707 1.5707"/>
+      <geometry>
+        <cylinder length="0.05" radius="0.1"/>
+      </geometry>
+    </collision>
+    <visual name='right2_wheel_visual'>
+      <origin xyz="0.0 0.0 0.0" rpy="0.0 1.5707 1.5707"/>
+      <geometry>
+        <cylinder length="0.05" radius="0.1"/>
+      </geometry>
+    </visual>
+  </link>
+  <joint type="continuous" name="right2_wheel_hinge">
+    <origin xyz="-0.25 -0.15 0" rpy="0 0 0"/>
+    <child link="right2_wheel"/>
+    <parent link="chassis"/>
+    <axis xyz="0 1 0" rpy="0 0 0"/>
+    <limit effort="10000" velocity="1000"/>
+    <dynamics damping="1.0" friction="1.0"/>
+  </joint>
+  <!-- Peripherals -->
   <link name='camera'>
     <inertial>
